Commit message: feat: integrate nav2 into launch file, optimize parameters, and add camera sensor urdf

File: urdf/robot.urdf (robot description, URDF)
Before this commit: robot diff_drive_robot, 6 links, 5 joints
Links:
- added link camera_link; collision box size=0.05 0.05 0.05; visual box size=0.05 0.05 0.05
Joints:
- added joint camera_joint: type fixed, parent base_link, child camera_link, origin xyz=0.2 0.0 0.1 rpy=0 0 0
